File: ADV728xM_EVAL_SMA-FFC_JETSON.sch (KiCad schematic (older format))
At the start: 13 parts, among them J1 142-0701-801, J2 142-0701-801, J3 142-0701-801, J4 142-0701-801, J5 Conn_01x04_Male, J6 Conn_01x04_Male, J7 Conn_01x02_Male, J8 Conn_01x02_Male, U1 1-84953-5, U2 NLSX5014DTR2G

Commit message: Add production release V1A
Connections:
- wire segments 62 -> 64
- no-connect marks 4 -> 2
Changed lines of the file:
@@
 Wire Wire Line
 	7375 5625 7375 5675
-NoConn ~ 8625 4525
-NoConn ~ 8625 4425
 Wire Wire Line
 	7375 1700 7375 1825
@@
 Wire Wire Line
 	7700 1600 7375 1600
+Wire Wire Line
+	8625 4425 7800 4425
+Text Label 7900 4425 0    50   ~ 0
+GPIO1_1V8
+Wire Wire Line
+	8625 4525 7800 4525
+Text Label 7900 4525 0    50   ~ 0
+GPIO0_1V8
 $EndSCHEMATC
