File: ADV728xM_EVAL_SMA-FFC_JETSON.kicad_pcb (KiCad board)
At the start: 2 copper layers, 13 parts, among them J1 142-0701-801, J2 142-0701-801, J3 142-0701-801, J4 142-0701-801, J5 Conn_01x04_Male, J6 Conn_01x04_Male, J7 Conn_01x02_Male, J8 Conn_01x02_Male, U1 1-84953-5, U2 NLSX5014DTR2G

Commit message: Add production release V1A
Connections:
- U1 pad 11: Net-(U1-Pad11) -> /GPIO1_1V8
- U1 pad 12: Net-(U1-Pad12) -> /GPIO0_1V8
Routing:
- net /GPIO1_1V8: track 16.3 -> 30.2 mm
- net /GPIO0_1V8: track 14.4 -> 27.8 mm
- net GND: track 25.7 -> 30.3 mm
- net /I2C_SDA: track 23.8 -> 23.2 mm
- net /I2C_SCL: track 27.0 -> 26.5 mm
- net /D0_P: vias 2 -> 3
- net /D0_N: vias 2 -> 3
- net /CLK_P: vias 2 -> 3
- net /CLK_N: vias 2 -> 3
Other:
- board outline added: 59.3 x 33.6 mm

Commit message: Move SMA connetors to back layer
Parts:
- J1, J2, J3, J4: moved to B.Cu
- turned J1 to 180 degrees
- turned J2 to 180 degrees
- turned J3 to 180 degrees
- turned J4 to 180 degrees
Routing:
- net /CLK_P: track 51.3 -> 54.1 mm, vias 3 -> 1
- net /D0_N: track 47.2 -> 49.9 mm, vias 3 -> 1
- net /D0_P: vias 3 -> 1
- net /CLK_N: vias 3 -> 1
